File: progcc_v3_main/procon_gcc_main_pcb.kicad_sch (KiCad schematic)
At the start: 107 parts, among them J1 Rumble, J2 Rumble, J3 To Button Board, J4 Conn_01x06_Female, J5 Conn_01x02_Pin, J9 USB_C_Receptacle, P1 Endpoint, Q1 Q_PMOS_GDS, Q2 Q_NMOS_GSD, Q3 Q_NMOS_GSD, Q4 BSS138, Q5 BSS138, Q6 BSS138, SW1 GL18_SW, SW2 GL18_SW, SW3 TS-1187A-B-A-B, SW4 TS35CA, T1 36-8730, T2 36-8730, T3 36-8730, T4 36-8730, U1 GH39F (Hall SOT23), U10 MCP3002, U11 ST_LSM6, U2 GH39F (Hall SOT23), U3 GH39F (Hall SOT23), U4 GH39F (Hall SOT23), U5 ST_LSM6, U6 RP2040, U7 LP3986-33B3F, U8 MCP3002, U9 W25Q128JVS, Y1 Crystal_GND3

Commit message: remove D3
Parts:
- removed D3: CUS08F30, Diode_SMD:D_SOD-323_HandSoldering, symbol progcc_v3:CUS08F30
- removed J1, J2: Rumble, progcc_v3:rumble_pins, symbol progcc_v3:Conn_01x02_Male
Connections:
- net +3V3: now also C4.1, TP13.1, U7.2 (VO)
Changed lines of the file:
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@@
   (junction (at 91.44 45.72) (diameter 0) (color 0 0 0 0)
   )
-  (junction (at 91.44 76.2) (diameter 0) (color 0 0 0 0)
-  )
   (junction (at 128.27 62.23) (diameter 0) (color 0 0 0 0)
   )
-  (junction (at 91.44 69.85) (diameter 0) (color 0 0 0 0)
-  )
   (junction (at 205.74 134.62) (diameter 0) (color 0 0 0 0)
   )
@@
   (junction (at 57.15 67.31) (diameter 0) (color 0 0 0 0)
   )
-  (junction (at 91.44 78.74) (diameter 0) (color 0 0 0 0)
-  )
   (junction (at 364.49 130.81) (diameter 0) (color 0 0 0 0)
   )
@@
   (junction (at 269.24 127) (diameter 0) (color 0 0 0 0)
   )
-  (junction (at 91.44 67.31) (diameter 0) (color 0 0 0 0)
-  )
   (junction (at 67.31 125.73) (diameter 0) (color 0 0 0 0)
   )
@@
     (stroke (width 0) (type default))
   )
-  (wire (pts (xy 91.44 76.2) (xy 92.71 76.2))
-    (stroke (width 0) (type default))
-  )
   (wire (pts (xy 238.76 66.04) (xy 241.3 66.04))
     (stroke (width 0) (type default))
@@
     (stroke (width 0) (type default))
   )
+  (wire (pts (xy 130.81 119.38) (xy 146.05 119.38))
+    (stroke (width 0) (type default))
+  )
   (wire (pts (xy 160.02 177.8) (xy 158.75 177.8))
     (stroke (width 0) (type default))
@@
     (stroke (width 0) (type default))
   )
-  (wire (pts (xy 146.05 119.38) (xy 143.51 119.38))
-    (stroke (width 0) (type default))
-  )
   (wire (pts (xy 392.43 118.11) (xy 394.97 118.11))
     (stroke (width 0) (type default))
@@
     (stroke (width 0) (type default))
   )
-  (wire (pts (xy 91.44 78.74) (xy 92.71 78.74))
-    (stroke (width 0) (type default))
-  )
   (wire (pts (xy 99.06 152.4) (xy 96.52 152.4))
     (stroke (width 0) (type default))
@@
     (stroke (width 0) (type default))
   )
-  (wire (pts (xy 91.44 69.85) (xy 92.71 69.85))
-    (stroke (width 0) (type default))
-  )
   (wire (pts (xy 149.86 26.67) (xy 130.81 26.67))
     (stroke (width 0) (type default))
@@
     (stroke (width 0) (type default))
   )
-  (wire (pts (xy 135.89 119.38) (xy 130.81 119.38))
-    (stroke (width 0) (type default))
-  )
   (polyline (pts (xy 170.18 90.17) (xy 285.75 90.17))
     (stroke (width 0) (type default))
@@
     (stroke (width 0) (type default))
   )
-  (wire (pts (xy 91.44 67.31) (xy 92.71 67.31))
-    (stroke (width 0) (type default))
-  )
   (wire (pts (xy 91.44 45.72) (xy 91.44 46.99))
     (stroke (width 0) (type default))
@@
     )
   )
-  (symbol (lib_id "progcc_v3:CUS08F30") (at 139.7 119.38 180) (unit 1)
-    (in_bom yes) (on_board yes) (dnp no)
-    (property "Reference" "D3" (at 139.7 114.3 0)
-      (effects (font (size 1.27 1.27)))
-    )
-    (property "Value" "CUS08F30" (at 139.7 116.84 0)
-      (effects (font (size 1.27 1.27)))
-    )
-    (property "Footprint" "Diode_SMD:D_SOD-323_HandSoldering" (at 139.7 114.3 0)
-      (effects (font (size 1.27 1.27)) hide)
-    )
-    (property "Datasheet" "${KIPRJMOD}/../progcc_v3_libs/docs/CUS08F30_datasheet_en_20140414.pdf" (at 139.7 111.76 0)
-      (effects (font (size 1.27 1.27)) hide)
-    )
-    (property "MPN" "CUS08F30" (at 139.7 119.38 0)
-      (effects (font (size 1.27 1.27)) hide)
-    )
-    (pin "1")
-    (pin "2")
-    (instances
-      (project "procon_gcc_main_pcb"
-        (path "/9ec9c1c0-f5f6-4920-ad47-c5d4aa989114"
-          (reference "D3") (unit 1)
-        )
-      )
-    )
-  )
-  (symbol (lib_id "progcc_v3:Conn_01x02_Male") (at 97.79 76.2 0) (mirror y) (unit 1)
-    (in_bom no) (on_board yes) (dnp yes)
-    (property "Reference" "J2" (at 103.378 71.12 0)
-      (effects (font (size 1.27 1.27)))
-    )
-    (property "Value" "Rumble" (at 99.314 71.374 0)
-      (effects (font (size 1.27 1.27)) hide)
-    )
-    (property "Footprint" "progcc_v3:rumble_pins" (at 97.79 76.2 0)
-      (effects (font (size 1.27 1.27)) hide)
-    )
-    (property "Datasheet" "~" (at 97.79 76.2 0)
-      (effects (font (size 1.27 1.27)) hide)
-    )
-    (pin "1")
-    (pin "2")
-    (instances
-      (project "procon_gcc_main_pcb"
-        (path "/9ec9c1c0-f5f6-4920-ad47-c5d4aa989114"
-          (reference "J2") (unit 1)
-        )
-      )
-    )
-  )
   (symbol (lib_id "Device:Q_PMOS_GSD") (at 119.38 35.56 0) (mirror x) (unit 1)
     (in_bom yes) (on_board yes) (dnp no)
@@
         )
       )
-    )
-  )
-  (symbol (lib_id "progcc_v3:Conn_01x02_Male") (at 97.79 67.31 0) (mirror y) (unit 1)
-    (in_bom no) (on_board yes) (dnp yes)
-    (property "Reference" "J1" (at 103.378 66.04 0)
-      (effects (font (size 1.27 1.27)))
-    )
-    (property "Value" "Rumble" (at 90.678 63.5 0)
-      (effects (font (size 1.27 1.27)) hide)
-    )
-    (property "Footprint" "progcc_v3:rumble_pins" (at 97.79 67.31 0)
-      (effects (font (size 1.27 1.27)) hide)
-    )
-    (property "Datasheet" "~" (at 97.79 67.31 0)
-      (effects (font (size 1.27 1.27)) hide)
-    )
-    (pin "1")
-    (pin "2")
-    (instances
-      (project "procon_gcc_main_pcb"
-        (path "/9ec9c1c0-f5f6-4920-ad47-c5d4aa989114"
-          (reference "J1") (unit 1)
-        )
-      )
