File: progcc_v3_main/procon_gcc_main_pcb.kicad_sch (KiCad schematic)
At the start: 104 parts, among them J3 To Button Board, J4 Conn_01x06_Female, J5 Conn_01x02_Pin, J9 USB_C_Receptacle, P1 Endpoint, Q1 Q_PMOS_GDS, Q2 Q_NMOS_GSD, Q3 Q_NMOS_GSD, Q4 BSS138, Q5 BSS138, Q6 BSS138, SW1 GL18_SW, SW2 GL18_SW, SW3 TS-1187A-B-A-B, SW4 TS35CA, T1 36-8730, T2 36-8730, T3 36-8730, T4 36-8730, U1 GH39F (Hall SOT23), U10 MCP3002, U11 ST_LSM6, U2 GH39F (Hall SOT23), U3 GH39F (Hall SOT23), U4 GH39F (Hall SOT23), U5 ST_LSM6, U6 RP2040, U7 LP3986-33B3F, U8 MCP3002, U9 W25Q128JVS, Y1 Crystal_GND3

Commit message: Update regulator
Parts:
- removed C2, C4: 2.2uF, Capacitor_SMD:C_0603_1608Metric, symbol Device:C
- removed TP13: TestPoint, TestPoint:TestPoint_Pad_D1.5mm, symbol Connector:TestPoint
- removed U7: LP3986-33B3F, Package_TO_SOT_SMD:SOT-23, symbol Regulator_Linear:AP2127N-3.3
- added C24: 100n, Capacitor_SMD:C_0201_0603Metric, symbol Device:C
- added C3: 10uF, Capacitor_SMD:C_0805_2012Metric, symbol Device:C
- added L5: 1.3A 2.2uH ±20% 80mΩ, Inductor_SMD:L_1008_2520Metric, symbol Device:L
- added R3: 100, Resistor_SMD:R_0201_0603Metric, symbol Device:R
- added U4: TPS630001RCR, hhl:VREG_V62_16624-01YE, symbol hhl:TPS63000DRCR
Connections:
- net +3V3: now also C3.1, U4.1 (VOUT), U4.10 (FB); no longer D2.1 (K)
- net GND: now also C24.1, C3.2, U4.11 (EP), U4.11_1 (EP), U4.11_2 (EP), U4.11_3 (EP), U4.11_4 (EP), U4.11_5 (EP), U4.11_6 (EP), U4.11_7 (EP), U4.11_8 (EP), U4.3 (PGND), U4.9 (GND)
- net +5V renamed +VCC
- net +VCC: now also D2.1 (K), R3.1, U4.5 (VIN)
- new net: C24.2, R3.2, U4.6 (EN), U4.7 (PS/SYNC), U4.8 (VINA)
- new net: L5.2, U4.2 (L2)
- new net: L5.1, U4.4 (L1)
Other:
- moved on the sheet: C3, C5, C6, D2, F2, J4, SW1, SW2, TP9, U5
